Commit message: added new p3dx file

File: src/p3dx/p3dx_description/urdf/pioneer3dx1.xacro (robot description, xacro)
@@ -18,5 +18,5 @@
 <robot name="pioneer3dx" xmlns:xacro="http://ros.org/wiki/xacro">
   <!-- import all gazebo-customization elements, including gazebo colors -->
-  <xacro:include filename="$(find p3dx_description)/urdf/pioneer3dx.gazebo" />
+  <xacro:include filename="$(find p3dx_description)/urdf/pioneer3dx1.gazebo" />
   <!-- import the pioneer 3dx's wheels -->
   <xacro:include filename="$(find p3dx_description)/urdf/pioneer3dx_wheel.xacro" />

File: src/p3dx/p3dx_description/urdf/pioneer3dx_wheel.xacro (robot description, xacro)
@@ -29,5 +29,5 @@
 					iyz="0" izz="0.011763977943" />
 			</inertial>
-			<visual >
+			<visual name="base_visual">
 				<origin xyz="0 0 0" rpy="0 0 0" />
 				<geometry name="pioneer_geom">
@@ -59,5 +59,5 @@
 					iyz="0" izz="0.011763977943" />
 			</inertial>
-			<visual>
+			<visual name="base_visual">
 				<origin xyz="0 0 0" rpy="0 0 0" />
 				<geometry name="pioneer_geom">
